File: feather_kicad/feather_multi_oled.sch (KiCad schematic (older format))
At the start: 71 parts, among them J1 Barrel_Jack_Switch, U1 feather, U10 SSD1309_transparent_oled, U11 SSD1309_transparent_oled, U12 SSD1309_transparent_oled, U13 MPU-6050, U2 SSD1309_transparent_oled, U3 SSD1309_transparent_oled, U4 SSD1309_transparent_oled, U5 SSD1309_transparent_oled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

Commit message: Added BOM
Parts:
- D1: Digikey Part No. NSVRB521S30T1G‎ -> NSVRB521S30T1GOSCT-ND
- LS1: Digikey Part No. (none) -> 445-2525-1-ND
- R10, R11, R17, R19, R2, R3, R4, R5, R6, R7, R8, R9: Digikey Part No. RMCF0805FG100K -> RMCF0805FG100KCT-ND
- U1: Digikey Part No. (none) -> 1528-2648-ND
- U10, U11, U12, U2, U3, U4, U5, U6, U8, U9: Digikey Part No. 609-62674-221121ALFCT-ND -> 609-1210-1-ND
Changed lines of the file:
@@
 F 2 "project_footprints:FCI_62674-241121ALF" H 16650 2650 60  0001 C CNN
 F 3 "" H 16650 2650 60  0001 C CNN
-F 4 "609-62674-221121ALFCT-ND" H 16650 2650 50  0000 C CNN "Digikey Part No."
+F 4 "609-1210-1-ND" H 16650 2650 50  0000 C CNN "Digikey Part No."
 	1    16650 2650
 	1    0    0    -1
@@
 F 2 "Diode_SMD:D_SOD-523" V 12600 1150 50  0001 C CNN
 F 3 "~" V 12600 1150 50  0001 C CNN
-F 4 "NSVRB521S30T1G‎" H 12600 1150 50  0001 C CNN "Digikey Part No."
+F 4 "NSVRB521S30T1GOSCT-ND" H 12600 1150 50  0001 C CNN "Digikey Part No."
 	1    12600 1150
 	0    1    1    0
@@
 F 2 "Resistor_SMD:R_0805_2012Metric" H 2650 7900 50  0001 C CNN
 F 3 "" H 2650 7900 50  0000 C CNN
-F 4 "RMCF0805FG100K" H 2650 7900 50  0001 C CNN "Digikey Part No."
+F 4 "RMCF0805FG100KCT-ND" H 2650 7900 50  0001 C CNN "Digikey Part No."
 	1    2650 7900
 	1    0    0    -1
@@
 F 2 "Resistor_SMD:R_0805_2012Metric" H 2500 8400 50  0001 C CNN
 F 3 "" H 2500 8400 50  0000 C CNN
-F 4 "RMCF0805FG100K" H 2500 8400 50  0001 C CNN "Digikey Part No."
+F 4 "RMCF0805FG100KCT-ND" H 2500 8400 50  0001 C CNN "Digikey Part No."
 	1    2500 8400
 	1    0    0    -1
@@
 F 2 "Adafruit_FeatherWing:PCB_FeatherWing" H 3500 2650 60  0001 C CNN
 F 3 "" H 3500 2650 60  0001 C CNN
+F 4 "1528-2648-ND" H 3500 2650 50  0001 C CNN "Digikey Part No."
 	1    3500 2650
 	1    0    0    -1
@@
 F 2 "Resistor_SMD:R_0805_2012Metric" H 11150 2800 50  0001 C CNN
 F 3 "~" H 11150 2800 50  0001 C CNN
-F 4 "RMCF0805FG100K" H 11150 2800 50  0001 C CNN "Digikey Part No."
+F 4 "RMCF0805FG100KCT-ND" H 11150 2800 50  0001 C CNN "Digikey Part No."
 	1    11150 2800
 	1    0    0    -1
@@
 F 2 "Resistor_SMD:R_0805_2012Metric" H 9950 2800 50  0001 C CNN
 F 3 "~" H 9950 2800 50  0001 C CNN
-F 4 "RMCF0805FG100K" H 9950 2800 50  0001 C CNN "Digikey Part No."
+F 4 "RMCF0805FG100KCT-ND" H 9950 2800 50  0001 C CNN "Digikey Part No."
 	1    9950 2800
 	1    0    0    -1
@@
 F 2 "Resistor_SMD:R_0805_2012Metric" H 10250 2800 50  0001 C CNN
 F 3 "~" H 10250 2800 50  0001 C CNN
-F 4 "RMCF0805FG100K" H 10250 2800 50  0001 C CNN "Digikey Part No."
+F 4 "RMCF0805FG100KCT-ND" H 10250 2800 50  0001 C CNN "Digikey Part No."
 	1    10250 2800
 	1    0    0    -1
@@
 F 2 "Resistor_SMD:R_0805_2012Metric" H 10550 2800 50  0001 C CNN
 F 3 "~" H 10550 2800 50  0001 C CNN
-F 4 "RMCF0805FG100K" H 10550 2800 50  0001 C CNN "Digikey Part No."
+F 4 "RMCF0805FG100KCT-ND" H 10550 2800 50  0001 C CNN "Digikey Part No."
 	1    10550 2800
 	1    0    0    -1
@@
 F 2 "Resistor_SMD:R_0805_2012Metric" H 10850 2800 50  0001 C CNN
 F 3 "~" H 10850 2800 50  0001 C CNN
-F 4 "RMCF0805FG100K" H 10850 2800 50  0001 C CNN "Digikey Part No."
+F 4 "RMCF0805FG100KCT-ND" H 10850 2800 50  0001 C CNN "Digikey Part No."
 	1    10850 2800
 	1    0    0    -1
@@
 F 2 "Resistor_SMD:R_0805_2012Metric" H 11450 2800 50  0001 C CNN
 F 3 "~" H 11450 2800 50  0001 C CNN
-F 4 "RMCF0805FG100K" H 11450 2800 50  0001 C CNN "Digikey Part No."
+F 4 "RMCF0805FG100KCT-ND" H 11450 2800 50  0001 C CNN "Digikey Part No."
 	1    11450 2800
 	1    0    0    -1
@@
 F 2 "Resistor_SMD:R_0805_2012Metric" H 11750 2800 50  0001 C CNN
 F 3 "~" H 11750 2800 50  0001 C CNN
-F 4 "RMCF0805FG100K" H 11750 2800 50  0001 C CNN "Digikey Part No."
+F 4 "RMCF0805FG100KCT-ND" H 11750 2800 50  0001 C CNN "Digikey Part No."
 	1    11750 2800
 	1    0    0    -1
@@
 F 2 "Resistor_SMD:R_0805_2012Metric" H 12050 2800 50  0001 C CNN
 F 3 "~" H 12050 2800 50  0001 C CNN
-F 4 "RMCF0805FG100K" H 12050 2800 50  0001 C CNN "Digikey Part No."
+F 4 "RMCF0805FG100KCT-ND" H 12050 2800 50  0001 C CNN "Digikey Part No."
 	1    12050 2800
 	1    0    0    -1
@@
 F 2 "Resistor_SMD:R_0805_2012Metric" H 12350 2800 50  0001 C CNN
 F 3 "~" H 12350 2800 50  0001 C CNN
-F 4 "RMCF0805FG100K" H 12350 2800 50  0001 C CNN "Digikey Part No."
+F 4 "RMCF0805FG100KCT-ND" H 12350 2800 50  0001 C CNN "Digikey Part No."
 	1    12350 2800
 	1    0    0    -1
@@
 F 2 "Resistor_SMD:R_0805_2012Metric" H 12650 2800 50  0001 C CNN
 F 3 "~" H 12650 2800 50  0001 C CNN
-F 4 "RMCF0805FG100K" H 12650 2800 50  0001 C CNN "Digikey Part No."
+F 4 "RMCF0805FG100KCT-ND" H 12650 2800 50  0001 C CNN "Digikey Part No."
 	1    12650 2800
 	1    0    0    -1
@@
 F 2 "project_footprints:FCI_62674-241121ALF" H 20350 2700 60  0001 C CNN
 F 3 "" H 20350 2700 60  0001 C CNN
-F 4 "609-62674-221121ALFCT-ND" H 20350 2700 50  0001 C CNN "Digikey Part No."
+F 4 "609-1210-1-ND" H 20350 2700 50  0001 C CNN "Digikey Part No."
 	1    20350 2700
 	1    0    0    -1
@@
 F 2 "project_footprints:FCI_62674-241121ALF" H 16650 6000 60  0001 C CNN
 F 3 "" H 16650 6000 60  0001 C CNN
-F 4 "609-62674-221121ALFCT-ND" H 16650 6000 50  0001 C CNN "Digikey Part No."
+F 4 "609-1210-1-ND" H 16650 6000 50  0001 C CNN "Digikey Part No."
 	1    16650 6000
 	1    0    0    -1
@@
 F 2 "project_footprints:FCI_62674-241121ALF" H 20350 6050 60  0001 C CNN
 F 3 "" H 20350 6050 60  0001 C CNN
-F 4 "609-62674-221121ALFCT-ND" H 20350 6050 50  0001 C CNN "Digikey Part No."
+F 4 "609-1210-1-ND" H 20350 6050 50  0001 C CNN "Digikey Part No."
 	1    20350 6050
 	1    0    0    -1
@@
 F 2 "project_footprints:FCI_62674-241121ALF" H 16650 9200 60  0001 C CNN
 F 3 "" H 16650 9200 60  0001 C CNN
-F 4 "609-62674-221121ALFCT-ND" H 16650 9200 50  0001 C CNN "Digikey Part No."
+F 4 "609-1210-1-ND" H 16650 9200 50  0001 C CNN "Digikey Part No."
 	1    16650 9200
 	1    0    0    -1
@@
 F 2 "project_footprints:FCI_62674-241121ALF" H 20350 9250 60  0001 C CNN
 F 3 "" H 20350 9250 60  0001 C CNN
-F 4 "609-62674-221121ALFCT-ND" H 20350 9250 50  0001 C CNN "Digikey Part No."
+F 4 "609-1210-1-ND" H 20350 9250 50  0001 C CNN "Digikey Part No."
 	1    20350 9250
 	1    0    0    -1
@@
 F 2 "project_footprints:FCI_62674-241121ALF" H 16650 12550 60  0001 C CNN
 F 3 "" H 16650 12550 60  0001 C CNN
-F 4 "609-62674-221121ALFCT-ND" H 16650 12550 50  0001 C CNN "Digikey Part No."
+F 4 "609-1210-1-ND" H 16650 12550 50  0001 C CNN "Digikey Part No."
 	1    16650 12550
 	1    0    0    -1
@@
 F 2 "project_footprints:FCI_62674-241121ALF" H 20350 12600 60  0001 C CNN
 F 3 "" H 20350 12600 60  0001 C CNN
-F 4 "609-62674-221121ALFCT-ND" H 20350 12600 50  0001 C CNN "Digikey Part No."
+F 4 "609-1210-1-ND" H 20350 12600 50  0001 C CNN "Digikey Part No."
 	1    20350 12600
 	1    0    0    -1
@@
 F 2 "project_footprints:FCI_62674-241121ALF" H 12550 5950 60  0001 C CNN
 F 3 "" H 12550 5950 60  0001 C CNN
-F 4 "609-62674-221121ALFCT-ND" H 12550 5950 50  0001 C CNN "Digikey Part No."
+F 4 "609-1210-1-ND" H 12550 5950 50  0001 C CNN "Digikey Part No."
 	1    12550 5950
 	1    0    0    -1
@@
 F 2 "project_footprints:FCI_62674-241121ALF" H 12550 9200 60  0001 C CNN
 F 3 "" H 12550 9200 60  0001 C CNN
-F 4 "609-62674-221121ALFCT-ND" H 12550 9200 50  0001 C CNN "Digikey Part No."
+F 4 "609-1210-1-ND" H 12550 9200 50  0001 C CNN "Digikey Part No."
 	1    12550 9200
 	1    0    0    -1
@@
 F 2 "Buzzer_Beeper:Buzzer_TDK_PS1240P02BT_D12.2mm_H6.5mm" H 4165 4300 50  0001 C CNN
 F 3 "~" H 4165 4300 50  0001 C CNN
+F 4 "445-2525-1-ND" H 4200 4350 50  0001 C CNN "Digikey Part No."
 	1    4200 4350
 	1    0    0    -1
